File: pcb_design/DoodleBot/doodlebot_project (schematic and pcb)/DoodleBot.kicad_sch (KiCad schematic)
At the start: 39 parts, among them J1 Conn_01x04, J2 Conn_01x04, J3 USB_B_Micro, J4 BUZZER_HEADERS, J5 LED_HEADERS, J6 MARKER_HEADERS, J7 ERASER_HEADERS, U1 ESP32-S3-WROOM-1

Commit message: Reorganized project structure
Parts:
- BOOT1, RESET1: footprint Button_Switch_SMD:Panasonic_EVQPUJ_EVQPUA -> Button_Switch_SMD:SW_SPST_PTS647_Sx38
Changed lines of the file:
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@@
 			)
 		)
-		(property "Footprint" "Button_Switch_SMD:Panasonic_EVQPUJ_EVQPUA"
+		(property "Footprint" "Button_Switch_SMD:SW_SPST_PTS647_Sx38"
 			(at 41.91 149.86 0)
 			(effects
@@
 			)
 		)
-		(property "Footprint" "Button_Switch_SMD:Panasonic_EVQPUJ_EVQPUA"
+		(property "Footprint" "Button_Switch_SMD:SW_SPST_PTS647_Sx38"
 			(at 54.61 149.86 0)
 			(effects
